File: KiCad/Shield_Gas_Sensor/Shield_Gas_Sensor_Arduino/Shield_Gas_Sensor_Arduino.sch (KiCad schematic (older format))
At the start: 17 parts, among them J1 CONN_01X08, J2 CONN_01X04_MALE, P1 Power, P2 Analog, P3 Digital, P4 Digital, P5 CONN_01X01, P6 CONN_01X01, P7 CONN_01X01, P8 CONN_01X01, SW1 SW_Push, U1 TL071

Commit message: routing not finished
Parts:
- removed J1: CONN_01X08, Connector_PinSocket_2.54mm:PinSocket_1x08_P2.54mm_Vertical, symbol Shield_Gas_Sensor_Arduino-rescue:CONN_01X08-conn
- removed J2: CONN_01X04_MALE, Connector_PinHeader_2.54mm:PinHeader_1x04_P2.54mm_Vertical, symbol Shield_Gas_Sensor_Arduino-rescue:CONN_01X04_MALE-conn
- removed SW1: SW_Push, Button_Switch_THT:SW_PUSH-12mm, symbol Switch:SW_Push
- added J1: Conn_01x04, Connector_JST:JST_PH_B4B-PH-K_1x04_P2.00mm_Vertical, symbol Connector_Generic:Conn_01x04
- added SW1: SW_Push_Dual, Button_Switch_THT:SW_TH_Tactile_Omron_B3F-10xx, symbol Switch:SW_Push_Dual
- added U2: RN2483_Breakout, Module_RN2483_Breakout:Module_RN2483_Breakout, symbol RN2483_Breakout:RN2483_Breakout
Connections:
- no-connect marks 5 -> 7
Changed lines of the file:
@@
 Text Label 8750 4150 0    50   ~ 0
 A0
-Text Label 3800 900  2    50   ~ 0
-Tx
-Text Label 3800 1000 2    50   ~ 0
-Rx
-Text Label 3800 1100 2    50   ~ 0
-CTS
-Text Label 3800 1200 2    50   ~ 0
-RTS
-Text Label 3800 1300 2    50   ~ 0
-RST
-Text Label 3800 1400 2    50   ~ 0
-3V3
-Text Label 3800 1500 2    50   ~ 0
-Vin
-$Comp
-L Shield_Gas_Sensor_Arduino-rescue:CONN_01X04_MALE-conn J2
-U 1 1 5BC58C8B
-P 2550 2400
-F 0 "J2" H 2656 2890 50  0000 C CNN
-F 1 "CONN_01X04_MALE" H 2656 2799 50  0000 C CNN
-F 2 "Connector_PinHeader_2.54mm:PinHeader_1x04_P2.54mm_Vertical" H 2550 2700 50  0001 C CNN
-F 3 "" H 2550 2700 50  0001 C CNN
-	1    2550 2400
-	1    0    0    -1
-$EndComp
 $Comp
 L power:GND #PWR0101
@@
 L power:+5V #PWR0102
 U 1 1 5BC58D87
-P 2850 2300
-F 0 "#PWR0102" H 2850 2150 50  0001 C CNN
-F 1 "+5V" V 2865 2428 50  0000 L CNN
-F 2 "" H 2850 2300 50  0001 C CNN
-F 3 "" H 2850 2300 50  0001 C CNN
-	1    2850 2300
+P 2850 2200
+F 0 "#PWR0102" H 2850 2050 50  0001 C CNN
+F 1 "+5V" V 2865 2328 50  0000 L CNN
+F 2 "" H 2850 2200 50  0001 C CNN
+F 3 "" H 2850 2200 50  0001 C CNN
+	1    2850 2200
 	0    1    1    0
 $EndComp
-Text Label 2850 2500 0    50   ~ 0
+Text Label 2850 2300 0    50   ~ 0
 NC
-Text Label 2850 2700 0    50   ~ 0
+Text Label 2850 2400 0    50   ~ 0
 A0
-$Comp
-L Shield_Gas_Sensor_Arduino-rescue:CONN_01X08-conn J1
-U 1 1 5BC598C8
-P 4000 1250
-F 0 "J1" H 4078 1291 50  0000 L CNN
-F 1 "CONN_01X08" H 4078 1200 50  0000 L CNN
-F 2 "Connector_PinSocket_2.54mm:PinSocket_1x08_P2.54mm_Vertical" H 4000 1250 50  0001 C CNN
-F 3 "" H 4000 1250 50  0001 C CNN
-	1    4000 1250
-	1    0    0    -1
-$EndComp
-$Comp
-L power:GND #PWR0103
-U 1 1 5BC63AB1
-P 3800 1600
-F 0 "#PWR0103" H 3800 1350 50  0001 C CNN
-F 1 "GND" V 3805 1472 50  0000 R CNN
-F 2 "" H 3800 1600 50  0001 C CNN
-F 3 "" H 3800 1600 50  0001 C CNN
-	1    3800 1600
-	0    1    1    0
-$EndComp
 $Comp
 L Device:Buzzer BZ1
@@
 	7700 2100 7700 2250
 $Comp
-L Switch:SW_Push SW1
-U 1 1 5BCE6F8A
-P 7550 4600
-F 0 "SW1" V 7504 4748 50  0000 L CNN
-F 1 "SW_Push" V 7595 4748 50  0000 L CNN
-F 2 "Button_Switch_THT:SW_PUSH-12mm" H 7550 4800 50  0001 C CNN
-F 3 "" H 7550 4800 50  0001 C CNN
-	1    7550 4600
-	0    1    1    0
-$EndComp
-$Comp
 L power:GND #PWR0105
 U 1 1 5BCE7069
@@
 Text Label 7550 4200 0    50   ~ 0
 Reset
-Wire Wire Line
-	7550 4200 7550 4400
-Wire Wire Line
-	7550 4800 7550 5000
 Text Label 10850 4800 0    50   ~ 0
 2
@@
 Wire Notes Line
 	6800 500  6800 6400
+$Comp
+L power:GND #PWR0103
+U 1 1 5BC63AB1
+P 5950 2050
+F 0 "#PWR0103" H 5950 1800 50  0001 C CNN
+F 1 "GND" V 5955 1922 50  0000 R CNN
+F 2 "" H 5950 2050 50  0001 C CNN
+F 3 "" H 5950 2050 50  0001 C CNN
+	1    5950 2050
+	1    0    0    -1
+$EndComp
+Text Label 5750 2050 3    50   ~ 0
+3V3
+Text Label 5650 2050 3    50   ~ 0
+RST
+Text Label 5550 2050 3    50   ~ 0
+RTS
+Text Label 5450 2050 3    50   ~ 0
+CTS
+Text Label 5350 2050 3    50   ~ 0
+Rx
+Text Label 5250 2050 3    50   ~ 0
+Tx
+$Comp
+L RN2483_Breakout:RN2483_Breakout U2
+U 1 1 5BD9E979
+P 5500 1800
+F 0 "U2" H 6028 2040 50  0000 L CNN
+F 1 "RN2483_Breakout" H 6028 1949 50  0000 L CNN
+F 2 "Module_RN2483_Breakout:Module_RN2483_Breakout" H 5550 2600 50  0001 C CNN
+F 3 "" H 5550 2600 50  0001 C CNN
+	1    5500 1800
+	1    0    0    -1
+$EndComp
+$Comp
+L Switch:SW_Push_Dual SW1
+U 1 1 5BDA4B30
+P 7550 4600
+F 0 "SW1" V 7504 4748 50  0000 L CNN
+F 1 "SW_Push_Dual" V 7595 4748 50  0000 L CNN
+F 2 "Button_Switch_THT:SW_TH_Tactile_Omron_B3F-10xx" H 7550 4800 50  0001 C CNN
+F 3 "" H 7550 4800 50  0001 C CNN
+	1    7550 4600
+	0    1    1    0
+$EndComp
+Wire Wire Line
+	7550 4200 7550 4400
+Wire Wire Line
+	7550 4800 7550 5000
+NoConn ~ 7350 4400
+NoConn ~ 7350 4800
+$Comp
+L Connector_Generic:Conn_01x04 J1
+U 1 1 5BDAAC5A
+P 2650 2200
+F 0 "J1" H 2570 2517 50  0000 C CNN
+F 1 "Conn_01x04" H 2570 2426 50  0000 C CNN
+F 2 "Connector_JST:JST_PH_B4B-PH-K_1x04_P2.00mm_Vertical" H 2650 2200 50  0001 C CNN
+F 3 "~" H 2650 2200 50  0001 C CNN
+	1    2650 2200
+	-1   0    0    -1
+$EndComp
 $EndSCHEMATC

Commit message: Routing final card
Parts:
- U2: symbol RN2483_Breakout:RN2483_Breakout -> Shield_Gas_Sensor_Arduino-rescue:RN2483_Breakout-RN2483_Breakout
Other:
- moved on the sheet: J1
Changed lines of the file:
@@
 L power:GND #PWR0101
 U 1 1 5BC58D11
-P 2850 2100
-F 0 "#PWR0101" H 2850 1850 50  0001 C CNN
-F 1 "GND" V 2855 1972 50  0000 R CNN
-F 2 "" H 2850 2100 50  0001 C CNN
-F 3 "" H 2850 2100 50  0001 C CNN
-	1    2850 2100
+P 2400 2600
+F 0 "#PWR0101" H 2400 2350 50  0001 C CNN
+F 1 "GND" V 2405 2472 50  0000 R CNN
+F 2 "" H 2400 2600 50  0001 C CNN
+F 3 "" H 2400 2600 50  0001 C CNN
+	1    2400 2600
 	0    -1   -1   0
 $EndComp
@@
 L power:+5V #PWR0102
 U 1 1 5BC58D87
-P 2850 2200
-F 0 "#PWR0102" H 2850 2050 50  0001 C CNN
-F 1 "+5V" V 2865 2328 50  0000 L CNN
-F 2 "" H 2850 2200 50  0001 C CNN
-F 3 "" H 2850 2200 50  0001 C CNN
-	1    2850 2200
+P 2400 2700
+F 0 "#PWR0102" H 2400 2550 50  0001 C CNN
+F 1 "+5V" V 2415 2828 50  0000 L CNN
+F 2 "" H 2400 2700 50  0001 C CNN
+F 3 "" H 2400 2700 50  0001 C CNN
+	1    2400 2700
 	0    1    1    0
 $EndComp
-Text Label 2850 2300 0    50   ~ 0
+Text Label 2400 2800 0    50   ~ 0
 NC
-Text Label 2850 2400 0    50   ~ 0
+Text Label 2400 2900 0    50   ~ 0
 A0
 $Comp
@@
 2
 Wire Notes Line
-	2200 1600 2200 2900
+	1750 2100 1750 3400
 Wire Notes Line
-	2200 2900 3300 2900
+	1750 3400 2850 3400
 Wire Notes Line
-	3300 2900 3300 1600
+	2850 3400 2850 2100
 Wire Notes Line
-	3300 1600 2200 1600
+	2850 2100 1750 2100
 Wire Notes Line
-	2200 1850 3300 1850
-Text Notes 2300 1750 0    50   ~ 0
+	1750 2350 2850 2350
+Text Notes 1850 2250 0    50   ~ 0
 Gaz sensor connector
 Text Label 7500 2250 3    60   ~ 0
@@
 Tx
 $Comp
-L RN2483_Breakout:RN2483_Breakout U2
+L Shield_Gas_Sensor_Arduino-rescue:RN2483_Breakout-RN2483_Breakout U2
 U 1 1 5BD9E979
 P 5500 1800
@@
 L Connector_Generic:Conn_01x04 J1
 U 1 1 5BDAAC5A
-P 2650 2200
-F 0 "J1" H 2570 2517 50  0000 C CNN
-F 1 "Conn_01x04" H 2570 2426 50  0000 C CNN
-F 2 "Connector_JST:JST_PH_B4B-PH-K_1x04_P2.00mm_Vertical" H 2650 2200 50  0001 C CNN
-F 3 "~" H 2650 2200 50  0001 C CNN
-	1    2650 2200
+P 2200 2700
+F 0 "J1" H 2120 3017 50  0000 C CNN
+F 1 "Conn_01x04" H 2120 2926 50  0000 C CNN
+F 2 "Connector_JST:JST_PH_B4B-PH-K_1x04_P2.00mm_Vertical" H 2200 2700 50  0001 C CNN
+F 3 "~" H 2200 2700 50  0001 C CNN
+	1    2200 2700
 	-1   0    0    -1
 $EndComp
