File: KiCad/Shield_Gas_Sensor/Shield_Gas_Sensor_Arduino/Shield_Gas_Sensor_Arduino.kicad_pcb (KiCad board)
At the start: 2 copper layers, 68.6 x 53.3 mm, 14 parts, among them J1 CONN_01X08, J2 CONN_01X04_MALE, P1 Power, P2 Analog, P3 Digital, P4 Digital, P5 CONN_01X01, P6 CONN_01X01, P7 CONN_01X01, P8 CONN_01X01, U1 TL071

Commit message: Routage PCB on Kicad
Parts:
- added BZ1: Buzzer, Buzzer_Beeper:Buzzer_12x9.5RM7.6, F.Cu at (140.2, 85.7)
- added D1: LED, LED_THT:LED_D5.0mm_IRGrey, F.Cu at (123.7, 85.7)
- added SW1: SW_Push, Button_Switch_THT:SW_PUSH-12mm, F.Cu at (116.1, 109.9)
- moved J2 31.8 mm to (169.4, 90.8), turned to 180 degrees
- moved J1 30.5 mm to (169.4, 112.4), turned to 270 degrees
- moved R1 21.6 mm to (168.1, 103.5), turned to 180 degrees
- moved U1 11.7 mm to (155.4, 87.0), turned to 90 degrees
- moved RV1 8.98 mm to (135.1, 95.9), turned to 270 degrees
- moved R2 8.52 mm to (172.0, 97.2)
Connections:
- R2 pad 1: Net-(R2-Pad1) -> /2
- U1 pad 6: Net-(R2-Pad1) -> /2
Routing:
- net GND: track 23.0 -> 148.9 mm, vias 0 -> 1
- net /Reset: track 0.00 -> 47.5 mm
- net /2: track 0.00 -> 40.8 mm
- net Net-(RV1-Pad2): track 7.05 -> 24.2 mm
- net /9(**): track 0.00 -> 15.8 mm
- net /A0: track 42.3 -> 53.5 mm
- net Net-(R2-Pad1): track 9.78 -> 0.00 mm
- net Net-(BZ1-Pad2): track 0.00 -> 6.37 mm
- net +5V: track 84.1 -> 78.2 mm
- net Net-(R1-Pad2): track 16.1 -> 19.4 mm
- net /Vin: track 13.8 -> 12.5 mm
Other:
- net class Default: clearance 0.2 -> 0.4; trace_width 0.25 -> 0.5; via_dia 0.6 -> 1.2; via_drill 0.4 -> 0.8
- rule trace_clearance: 0.2 -> 0.4

Commit message: routing not finished
Parts:
- removed J2: CONN_01X04_MALE, Connector_PinHeader_2.54mm:PinHeader_1x04_P2.54mm_Vertical
- added U2: RN2483_Breakout, Module_RN2483_Breakout:Module_RN2483_Breakout, F.Cu at (117.3, 111.1)
- J1: value CONN_01X08 -> Conn_01x04; footprint Connector_PinSocket_2.54mm:PinSocket_1x08_P2.54mm_Vertical -> Connector_JST:JST_PH_B4B-PH-K_1x04_P2.00mm_Vertical
- SW1: value SW_Push -> SW_Push_Dual; footprint Button_Switch_THT:SW_PUSH-12mm -> Button_Switch_THT:SW_TH_Tactile_Omron_B3F-10xx
- moved D1 30.6 mm to (154.2, 88.3)
- moved R2 14.5 mm to (168.1, 111.1)
- moved U1 14.5 mm to (159.3, 101.0)
- moved SW1 14.5 mm to (127.5, 118.7)
- moved R1 13.7 mm to (156.7, 111.1)
- moved RV1 11.7 mm to (127.5, 104.8), turned to 0 degrees
- moved BZ1 6.84 mm to (146.6, 88.3)
- moved J1 6.35 mm to (175.8, 112.4), turned to 90 degrees
Connections:
- J1 pad 1: /Tx -> GND
- J1 pad 2: /Rx -> +5V
- J1 pad 3: /CTS -> /NC
- J1 pad 4: /RTS -> /A0
Routing:
- net GND: track 148.9 -> 28.4 mm, vias 1 -> 0
- net +5V: track 78.2 -> 0.00 mm
- net /A0: track 53.5 -> 0.00 mm
- net /Reset: track 47.5 -> 0.00 mm
- net /2: track 40.8 -> 0.00 mm
- net Net-(RV1-Pad2): track 24.2 -> 0.00 mm
- net Net-(R1-Pad2): track 19.4 -> 0.00 mm
- net /9(**): track 15.8 -> 0.00 mm
- net /Vin: track 12.5 -> 0.00 mm
- net Net-(BZ1-Pad2): track 6.37 -> 0.00 mm
- removed copper zone on B.Cu, net GND
